File: hardware/room-sensor/pcb/RoomSensor-MainPlate/RoomSensor-MainPlate.kicad_pcb (KiCad board)
At the start: 4 copper layers, 33 x 58 mm, 10 parts

Commit message: PCB Design
Parts:
- removed Audio: ES8311 + NS4150B, Connector_PinSocket_2.54mm:PinSocket_1x10_P2.54mm_Vertical
- removed B-Data: Backplate Data, Connector_JST:JST_XH_B6B-XH-A_1x06_P2.50mm_Vertical
- removed B_Power: Backplate Power, Connector_JST:JST_XH_B4B-XH-A_1x04_P2.50mm_Vertical
- removed Climate: ENS160 + AHT20, Connector_PinSocket_2.54mm:PinSocket_1x08_P2.54mm_Vertical
- removed ESP: ESP-POE2, Connector_PinSocket_2.54mm:PinSocket_2x13_P2.54mm_Vertical
- removed GPIO: GPIO, TerminalBlock_Phoenix:TerminalBlock_Phoenix_MPT-0,5-7-2.54_1x07_P2.54mm_Horizontal
- removed LED: LED Connector, TerminalBlock_Phoenix:TerminalBlock_Phoenix_MPT-0,5-4-2.54_1x04_P2.54mm_Horizontal
- removed Light: BH1750, Connector_PinSocket_2.54mm:PinSocket_1x05_P2.54mm_Vertical
- removed Motion: Dfrobot C4002, Connector_PinSocket_2.54mm:PinSocket_1x05_P2.54mm_Vertical
- removed Power: Power, TerminalBlock_Phoenix:TerminalBlock_Phoenix_MPT-0,5-4-2.54_1x04_P2.54mm_Horizontal
- added A1: ES8311 + NS4150B, room-sensor:ES8311 + NS4150B Connector, F.Cu at (85.0, 81.5)
- added C1: LED Connector, TerminalBlock_Phoenix:TerminalBlock_Phoenix_MPT-0,5-4-2.54_1x04_P2.54mm_Horizontal, F.Cu at (90.1, 49.0)
- added C2: Power, TerminalBlock_Phoenix:TerminalBlock_Phoenix_MPT-0,5-4-2.54_1x04_P2.54mm_Horizontal, B.Cu at (78.0, 71.1)
- added C3: GPIO, TerminalBlock_Phoenix:TerminalBlock_Phoenix_MPT-0,5-7-2.54_1x07_P2.54mm_Horizontal, B.Cu at (78.0, 59.2)
- added E1: ESP-POE2, Connector_PinSocket_2.54mm:PinSocket_2x13_P2.54mm_Vertical, B.Cu at (89.5, 55.0)
- added J1: B2B_Connector, room-sensor:B2B Connector, B.Cu at (74.5, 89.6)
- added S1: Dfrobot C4002, room-sensor:DFRobot C4002 Connector, F.Cu at (97.0, 77.0)
- added S2: BH1750, room-sensor:BH1750, F.Cu at (92.0, 90.0)
- added S3: ENS160 + AHT20, room-sensor:ENS160 + AHT20 Connector, F.Cu at (97.0, 48.0)
Routing:
- net Net-(C1-DIn): track 0.00 -> 40.9 mm
- net /+12/24V: track 75.7 -> 38.1 mm
- net /+5V: track 126.3 -> 89.2 mm
- net /SDA: track 83.0 -> 49.3 mm
- net /+3.3V: track 56.5 -> 36.3 mm
- net /E_TX: track 43.2 -> 29.7 mm
- net /LED: track 20.0 -> 33.0 mm
- net /E_RX: track 38.9 -> 49.8 mm
- net /A_MCLK: track 17.6 -> 28.1 mm
- net Net-(C1-DOut): track 9.22 -> 0.00 mm
- net /GND: track 95.9 -> 87.0 mm
- net /SCL: track 67.8 -> 59.6 mm
- net /A_DO: track 42.3 -> 50.3 mm
- net /A_LRCLK: track 35.0 -> 42.0 mm
- net /A_BCLK: track 22.8 -> 28.4 mm
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Other:
- board size 33 x 58 mm -> 31 x 54 mm
