File: hardware/pcb/RoomSensor-MainPlate/RoomSensor-MainPlate.kicad_sch (KiCad schematic)
At the start: 9 parts, among them J1 B2B_Connector

Commit message: hardware: move footprint/symbol libs into pcb/, update KiCad project settings
Move room-sensor.pretty/ and room-sensor.kicad_sym into hardware/pcb/ so all
PCB design files live under one directory. Also picks up KiCad project edits:
BOM preset config and pin_to_pin ERC rule change to error on both plates.

Co-Authored-By: Claude Sonnet 4.6 <noreply@anthropic.com>
Parts:
- A1: MPN 61301011821 -> PM254-1-10-Z-8.5
- C1, C2: MPN 1725672 -> KF128-2.54-4P
- C3: MPN 1725708 -> KF128-2.54-7P
- E1: MPN 61302621821 -> C64320
- J1: MPN (none) -> MTB10-10S
- S1, S2: MPN 61300511821 -> C50950
- S3: MPN 61300811821 -> C27438
Changed lines of the file:
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@@
+			)
+		)
+		(property "MPN" "MTB10-10S"
+			(at 111.76 147.32 0)
+			(hide yes)
+			(show_name no)
+			(do_not_autoplace no)
+			(effects
+				(font
+					(size 1.27 1.27)
+				)
+			)
+		)
+		(property "LCSC" ""
+			(at 111.76 147.32 0)
+			(hide yes)
+			(show_name no)
+			(do_not_autoplace no)
+			(effects
+				(font
+					(size 1.27 1.27)
+				)
 			)
 		)
@@
 			)
 		)
-		(property "MPN" "61300811821"
+		(property "MPN" "C27438"
+			(at 111.76 78.74 0)
+			(hide yes)
+			(show_name no)
+			(do_not_autoplace no)
+			(effects
+				(font
+					(size 1.27 1.27)
+				)
+			)
+		)
+		(property "LCSC" ""
 			(at 111.76 78.74 0)
 			(hide yes)
@@
 			)
 		)
-		(property "MPN" "1725708"
+		(property "MPN" "KF128-2.54-7P"
+			(at 113.03 128.27 0)
+			(hide yes)
+			(show_name no)
+			(do_not_autoplace no)
+			(effects
+				(font
+					(size 1.27 1.27)
+				)
+			)
+		)
+		(property "LCSC" ""
 			(at 113.03 128.27 0)
 			(hide yes)
@@
 			)
 		)
-		(property "MPN" "61301011821"
+		(property "MPN" "PM254-1-10-Z-8.5"
+			(at 111.76 102.87 0)
+			(hide yes)
+			(show_name no)
+			(do_not_autoplace no)
+			(effects
+				(font
+					(size 1.27 1.27)
+				)
+			)
+		)
+		(property "LCSC" ""
 			(at 111.76 102.87 0)
 			(hide yes)
@@
 			)
 		)
-		(property "MPN" "61300511821"
+		(property "MPN" "C50950"
+			(at 111.76 46.99 0)
+			(hide yes)
+			(show_name no)
+			(do_not_autoplace no)
+			(effects
+				(font
+					(size 1.27 1.27)
+				)
+			)
+		)
+		(property "LCSC" ""
 			(at 111.76 46.99 0)
 			(hide yes)
@@
 			)
 		)
-		(property "MPN" "61302621821"
+		(property "MPN" "C64320"
+			(at 46.99 101.6 0)
+			(hide yes)
+			(show_name no)
+			(do_not_autoplace no)
+			(effects
+				(font
+					(size 1.27 1.27)
+				)
+			)
+		)
+		(property "LCSC" ""
 			(at 46.99 101.6 0)
 			(hide yes)
@@
 			)
 		)
-		(property "MPN" "61300511821"
+		(property "MPN" "C50950"
+			(at 111.76 62.23 0)
+			(hide yes)
+			(show_name no)
+			(do_not_autoplace no)
+			(effects
+				(font
+					(size 1.27 1.27)
+				)
+			)
+		)
+		(property "LCSC" ""
 			(at 111.76 62.23 0)
 			(hide yes)
@@
 			)
 		)
-		(property "MPN" "1725672"
+		(property "MPN" "KF128-2.54-4P"
+			(at 113.03 175.26 0)
+			(hide yes)
+			(show_name no)
+			(do_not_autoplace no)
+			(effects
+				(font
+					(size 1.27 1.27)
+				)
+			)
+		)
+		(property "LCSC" ""
 			(at 113.03 175.26 0)
 			(hide yes)
@@
 			)
 		)
-		(property "MPN" "1725672"
+		(property "MPN" "KF128-2.54-4P"
 			(at 113.03 161.29 0)
 			(hide yes)
+			(show_name no)
+			(do_not_autoplace no)
+			(effects
+				(font
+					(size 1.27 1.27)
+				)
+			)
+		)
+		(property "LCSC" ""
+			(at 113.03 161.29 0)
+			(hide yes)
