File: hardware/pcb/RoomSensor-MainPlate/RoomSensor-MainPlate.kicad_sch (KiCad schematic)
At the start: 9 parts, among them J1 B2B_Connector

Commit message: Updated PCB to Rev 2 and 3
Parts:
- removed A1: ES8311 + NS4150B, room-sensor:ES8311 + NS4150B Connector, symbol Connector:Conn_01x10_Socket
- removed C2: Power, TerminalBlock_Phoenix:TerminalBlock_Phoenix_MPT-0,5-4-2.54_1x04_P2.54mm_Horizontal, symbol Connector:Screw_Terminal_01x04
- removed C3: GPIO, TerminalBlock_Phoenix:TerminalBlock_Phoenix_MPT-0,5-7-2.54_1x07_P2.54mm_Horizontal, symbol Connector:Screw_Terminal_01x07
- added J2: GPIO, Connector_IDC:IDC-Header_2x05_P2.54mm_Vertical, symbol room-sensor:B2B_Connector
Connections:
- net A_LRCLK is gone; now on net SDA: E1.25 (GPIO13)
- net A_MCLK is gone; now on net E_RX: E1.13 (GPIO1)
- net +12/24V: now also J2.5 (+24/12V)
- net +3.3V: now also S2.5 (VCC), S3.2 (3V3), J2.1 (+3.3V)
- net +5V: now also J2.3 (+5V); no longer S2.5 (VCC), S3.1 (Vin)
- net E_RX: no longer E1.10 (GPI39)
- net E_TX: now also E1.17 (GPIO3); no longer E1.18 (GPIO33)
- net GND: now also J2.7 (GND)
- net M_RX: now also E1.14 (GPI35); no longer E1.12 (GPI36)
- net M_TX: now also E1.19 (GPIO4); no longer E1.15 (GPIO2)
- net SCL: now also E1.18 (GPIO33); no longer E1.17 (GPIO3)
- net SDA: no longer E1.19 (GPIO4)
- net at E1.16 (GPI34): now also J2.10 (GPI34_(10k/BUT))
- net A_BCLK: no longer names the net of E1.21 (GPIO5)
- net A_BCLK: now also J2.4 (GPIO5_(10k))
- net A_DI: no longer names the net of J1.9 (IO_INT)
- net A_DI: now also E1.12 (GPI36); no longer E1.24 (GPIO15)
- net A_DO: no longer names the net of E1.26 (GPIO14)
- net A_DO: now also J2.6 (GPIO14)
- new net: E1.10 (GPI39), J2.9 (GPI39_(PWR_Sense))
- new net: E1.15 (GPIO2), J2.2 (GPIO2_(2.2k))
- new net: E1.24 (GPIO15), J2.8 (GPIO15_(10k))
