File: hardware/pcb/RoomSensor-MainPlate/RoomSensor-MainPlate.kicad_pcb (KiCad board)
At the start: 4 copper layers, 31 x 54 mm, 9 parts, among them J1 B2B_Connector

Commit message: hardware: move footprint/symbol libs into pcb/, update KiCad project settings
Move room-sensor.pretty/ and room-sensor.kicad_sym into hardware/pcb/ so all
PCB design files live under one directory. Also picks up KiCad project edits:
BOM preset config and pin_to_pin ERC rule change to error on both plates.

Co-Authored-By: Claude Sonnet 4.6 <noreply@anthropic.com>
Other:
- board text added: "universal-home-sensor MainPlate, Rev. 1 Frank Steiler, 2026"

Commit message: hardware: back plate mounting holes + EX2 routing, plot settings cleanup
BackPlate: add four M3 mounting holes, re-place EX2 (I2S External) and
route the remaining nets (+26 track segments, 7 new schematic wires).
MainPlate: switch plot output to a repo-relative directory instead of a
local Desktop path, add board outline/keepout drawings.

Co-Authored-By: Claude Opus 5 (1M context) <noreply@anthropic.com>
Other:
- board text added: "10x10mm"
Changed lines of the file:
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@@
 		(filling no)
 		(pcbplotparams
-			(layerselection 0x00000000_00000000_55555555_5755f5ff)
-			(plot_on_all_layers_selection 0x00000000_00000000_00000000_00000000)
+			(layerselection 0x00000000_00000000_55555555_555555a0)
+			(plot_on_all_layers_selection 0x00000000_00000000_00000000_02020000)
 			(disableapertmacros no)
 			(usegerberextensions no)
@@
 			(crossoutdnponfab yes)
 			(subtractmaskfromsilk no)
-			(outputformat 1)
+			(outputformat 5)
 			(mirror no)
 			(drillshape 0)
 			(scaleselection 1)
-			(outputdirectory "/Users/franksteiler/Desktop/")
+			(outputdirectory "./")
 		)
 	)
@@
 		(sheetname "/")
 		(sheetfile "RoomSensor-MainPlate.kicad_sch")
-		(units
-			(unit
-				(name "A")
-				(pins "1" "3" "5" "7" "9" "11" "13" "15" "17" "19" "21" "23" "25" "2"
-					"4" "6" "8" "10" "12" "14" "16" "18" "20" "22" "24" "26"
-				)
-			)
-		)
 		(attr through_hole)
 		(duplicate_pad_numbers_are_jumpers no)
@@
 			(layer "B.SilkS")
 		)
+		(fp_rect
+			(start -33 -51.5)
+			(end -17 -75)
+			(stroke
+				(width 0.1)
+				(type default)
+			)
+			(fill no)
+			(layer "Dwgs.User")
+		)
+		(fp_circle
+			(center 1 9.76)
+			(end 2.5 9.76)
+			(stroke
+				(width 0.1)
+				(type default)
+			)
+			(fill no)
+			(layer "Dwgs.User")
+		)
+		(fp_circle
+			(center 1 -40.24)
+			(end 2.5 -40.24)
+			(stroke
+				(width 0.1)
+				(type default)
+			)
+			(fill no)
+			(layer "Dwgs.User")
+		)
+		(fp_circle
+			(center -51 9.76)
+			(end -49.5 9.76)
+			(stroke
+				(width 0.1)
+				(type default)
+			)
+			(fill no)
+			(layer "Dwgs.User")
+		)
+		(fp_circle
+			(center -51 -40.24)
+			(end -49.5 -40.24)
+			(stroke
+				(width 0.1)
+				(type default)
+			)
+			(fill no)
+			(layer "Dwgs.User")
+		)
 		(fp_line
 			(start 1.77 1.77)
@@
 		)
 	)
+	(gr_rect
+		(start 60 32)
+		(end 70 42)
+		(stroke
+			(width 0.1)
+			(type default)
+		)
+		(fill no)
+		(layer "Dwgs.User")
+	)
 	(gr_line
 		(start 115 124)
@@
 			)
 			(justify left bottom)
+		)
+	)
+	(gr_text "10x10mm"
+		(at 61.5 37 0)
+		(layer "Dwgs.User")
+		(effects
+			(font
+				(size 1 1)
+				(thickness 0.15)
+			)
+			(justify left bottom)
