File: hardware/pcb/RoomSensor-BackPlate/RoomSensor-BackPlate.kicad_pcb (KiCad board)
At the start: 4 copper layers, 82 x 61 mm, 20 parts, among them U1 PCF8574P

Commit message: Updated PCB to Rev 2 and 3
Parts:
- removed JP1, JP2, JP3, JP4, JP5, JP6: SolderJumper_2_Open, Jumper:SolderJumper-2_P1.3mm_Open_Pad1.0x1.5mm
- removed REF** (x4): MountingHole_3.2mm_M3, MountingHole:MountingHole_3.2mm_M3
- R1, R2, R3: value Relay -> 2-Way Relay Module
- moved EX1 22.3 mm to (102.0, 109.5), turned to 0 degrees
- moved EX3 18.6 mm to (104.0, 95.5)
- moved R1 10.7 mm to (129.0, 85.2)
- moved EX2 10.3 mm to (114.5, 109.5), turned to 0 degrees
- moved C1 7.48 mm to (129.0, 99.9)
- moved U1 1.38 mm to (138.8, 81.1)
Connections:
- C1 pad 1: Net-(C1-+3.3V) -> /+3.3V
- C1 pad 10: /LED Bus -> Net-(C1-LED)
- C1 pad 9: /GPIO15 -> Net-(C1-IO_INT)
- EX1 pad 1: Net-(EX1-V+) -> Net-(C1-+24/12V)
- EX1 pad 2: /LED Bus -> /+5V
- EX1 pad 3: /GPIO15 -> Net-(C1-LED)
- EX2 pad 1: Net-(EX2-V+) -> /+3.3V
- R1 pad 1: /+5V -> /+3.3V
- R2 pad 1: /+5V -> /+3.3V
- R3 pad 1: /+5V -> /+3.3V
- U1 pad 13: unconnected-(U1-~{INT}-Pad13) -> Net-(C1-IO_INT)
- U1 pad 16: /+5V -> /+3.3V
Routing:
- net /+3.3V: track 0.00 -> 104.7 mm
- net Net-(C1-IO_INT): track 0.00 -> 43.8 mm
- net Net-(C1-+3.3V): track 41.3 -> 0.00 mm, vias 2 -> 0
- net /E-GPIO5: track 102.1 -> 65.2 mm
- net Net-(C1-Energy_TX): track 85.2 -> 57.1 mm
- net /LED Bus: track 28.0 -> 0.00 mm
- net /E-GPIO7: track 82.7 -> 56.0 mm
- net Net-(C1-LED): track 0.00 -> 26.7 mm
- net /+5V: track 167.0 -> 193.2 mm, vias 2 -> 0
- net /GPIO15: track 24.4 -> 0.00 mm
- net Net-(C1-Energy_RX): track 81.4 -> 57.1 mm
- net /E-GPIO6: track 89.6 -> 67.3 mm
- net Net-(EX2-V+): track 21.1 -> 0.00 mm, vias 1 -> 0
- net Net-(EX1-V+): track 18.2 -> 0.00 mm, vias 1 -> 0
- net Net-(C1-+24/12V): track 17.0 -> 31.7 mm, vias 2 -> 0
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Other:
- board size 82 x 61 mm -> 82 x 56 mm
- board text added: "+24/12V"
- board text added: "MainPlate"
- board text added: "universal-home-sensor BackPlate, Rev. 3 Frank Steiler, 2026"
- board text removed: "10x10mm"
- board text removed: "12/24V"
- board text removed: "3.3V"
- board text removed: "5V"
- board text removed: "EX1"
- board text removed: "GPIO15"
- board text removed: "LEDOut"
- board text removed: "Only 1 pad!"
- board text removed: "SCL"
- board text removed: "SDA"
- board text removed: "V+"
- board text removed: "universal-home-sensor BackPlate, Rev. 2a Frank Steiler, 2026"
