File: hardware/pcb/RoomSensor-BackPlate/RoomSensor-BackPlate.kicad_sch (KiCad schematic)
At the start: 16 parts, among them U1 PCF8574P

Commit message: Updated PCB to Rev 2 and 3
Parts:
- removed JP1, JP2, JP3, JP4, JP5, JP6: SolderJumper_2_Open, Jumper:SolderJumper-2_P1.3mm_Open_Pad1.0x1.5mm, symbol Jumper:SolderJumper_2_Open
- removed R1, R2, R3: Relay, room-sensor:2-way Relay Connector, symbol Connector_Generic:Conn_01x04
- added R1, R2, R3: 2-Way Relay Module, room-sensor:2-way Relay Connector, symbol room-sensor:5V_2_Relay_Module
Connections:
- net +5V: now also EX1.2 (+5V), R1.7 (RY-VCC), R2.7 (RY-VCC), R3.7 (RY-VCC); no longer U1.16 (VDD)
- net E-GPIO0: now also R3.2 (IO2)
- net E-GPIO1: now also R3.3 (IO1)
- net E-GPIO2: now also R2.2 (IO2)
- net E-GPIO3: now also R2.3 (IO1)
- net E-GPIO4: now also R1.2 (IO2)
- net E-GPIO5: now also R1.3 (IO1)
- net GND: now also R1.4 (GND), R2.4 (GND), R3.4 (GND)
- net +3.3V: now reaches C1.1 (+3.3V)
- net +3.3V: now also EX2.1 (+3.3V), U1.16 (VDD), R1.1 (VCC), R2.1 (VCC), R3.1 (VCC)
- net at C1.5 (+24/12V): now also EX1.1 (+24/12V)
- net at U1.13 (~{INT}): now also C1.9 (IO_INT)
- net GPIO15: no longer names the net of EX1.3 (LED-Bus)
- net GPIO15: now also C1.10 (LED); no longer C1.9 (GPIO15)
- removed net LED Bus: C1.10 (LED), EX1.2 (LED_Bus)
Other:
- moved on the sheet: EX2, EX3
